File: Nucleo.kicad_sch (KiCad schematic)
At the start: 1 part, among them U12 NUCLEO-H755ZIQ

Commit message: PCB layout first commit, minor fix in schematic
Connections:
- net SDMMC_CK: now reaches U12.10 (PC12)
- net SDMMC_CMD: now reaches U12.12 (PD2)
- net DETECT_SD: now reaches U12.14 (PG10)
- net TO_ADC1: now reaches U12.17 (PA3)
- net TO_ADC2: now reaches U12.19 (PC0)
- net SDMMC_D0: now reaches U12.2 (PC8)
- net SDMMC_D1: now reaches U12.4 (PC9)
- net SDMMC_D2: now reaches U12.6 (PC10)
- net SDMMC_D3: now reaches U12.8 (PC11)
- no-connect marks 0 -> 81

Commit message: New STM footprint, changed PCB layout, added pin connector
Parts:
- removed U12: NUCLEO-H755ZIQ, Uklad_wzmacniaczy_footprints:Nucleo-H755ZIQ, symbol Amplifier_circuit:Nucleo-H755ZIQ
- added C35, C42, C43: 10u, Capacitor_SMD:C_0603_1608Metric_Pad1.08x0.95mm_HandSolder, symbol Device:C
- added C36: 1u, Capacitor_SMD:C_0603_1608Metric_Pad1.08x0.95mm_HandSolder, symbol Device:C
- added C37: 10p, Capacitor_SMD:C_0603_1608Metric_Pad1.08x0.95mm_HandSolder, symbol Device:C
- added C38, C39, C40: 22u, Capacitor_SMD:C_0603_1608Metric_Pad1.08x0.95mm_HandSolder, symbol Device:C
- added C41: 10n, Capacitor_SMD:C_0603_1608Metric_Pad1.08x0.95mm_HandSolder, symbol Device:C
- added D1: LED, LED_SMD:LED_0805_2012Metric_Pad1.15x1.40mm_HandSolder, symbol Device:LED
- added L2: 1u, Uklad_wzmacniaczy_footprints:IND_SPM6530T-1R0M120, symbol Device:L
- added R17: 1M, Resistor_SMD:R_0603_1608Metric_Pad0.98x0.95mm_HandSolder, symbol Device:R
- added R18: 332k, Resistor_SMD:R_0603_1608Metric_Pad0.98x0.95mm_HandSolder, symbol Device:R
- added R19: 2k, Resistor_SMD:R_0603_1608Metric_Pad0.98x0.95mm_HandSolder, symbol Device:R
- added R20: 41.2k, Resistor_SMD:R_0603_1608Metric_Pad0.98x0.95mm_HandSolder, symbol Device:R
- added U13: Nucleo-H755ZIQ-Morpho, Uklad_wzmacniaczy_footprints:Nucleo-H755ZIQ-Morpho, symbol Amplifier_circuit:Nucleo-H755ZIQ-Morpho
- added U14: TPS61236PRWLR, Uklad_wzmacniaczy_footprints:RWL0009A, symbol Amplifier_circuit:TPS61236PRWLR
- added U15: LD1117S50TR_SOT223, Package_TO_SOT_SMD:SOT-223-3_TabPin2, symbol Regulator_Linear:LD1117S50TR_SOT223
Connections:
- net GND: now also C35.2, C36.2, C38.2, C39.2, C40.2, C41.2, R18.1, R19.1, R20.1, U14.1 (PGND), U14.5 (AGND)
- net GNDA: now also C42.2, C43.2, U15.1 (GND)
- net SDMMC_CK: now also U13.1.03 (PC12)
- net SDMMC_CMD: now also U13.1.04 (PD2)
- net SDMMC_D0: now also U13.2.02 (PC8)
- net SDMMC_D1: now also U13.2.01 (PC9)
- net SDMMC_D2: now also U13.1.01 (PC10)
- net SDMMC_D3: now also U13.1.02 (PC11)
- net TO_ADC1: now also U13.1.28 (PA0)
- net TO_ADC2: now also U13.1.32 (PA4)
- new net: C37.2, R17.1, R18.2, U14.6 (FB)
- new net: D1.1 (K), R19.2
- new net: L2.2, U14.2 (SW)
- new net +3.3V: C43.1, U15.2 (VO)
- new net +5V: C37.1, C38.1, C39.1, C40.1, C42.1, D1.2 (A), R17.2, U14.9 (VOUT), U15.3 (VI)
- new net +BATT: C35.1, C36.1, L2.1, U14.3 (VIN), U14.7 (EN)
- new net CC: C41.1, R20.2, U14.4 (CC)
- new net SIG_1: U13.1.09 (PF6)
- new net SIG_2: U13.1.11 (PF7)
- new net SIG_3: U13.1.38 (PC0)
- new net SIG_4: U13.1.35 (PC2)
- new net SIG_5: U13.1.37 (PC3)
- no-connect marks 81 -> 19
Other:
- note added: "[x] SIG PONUMEROWAĆ ODPOWIEDNIO Z DOKUMENTACJĄ [x] DODAĆ PIN T0_ADC2 [x] SPRAWDZIĆ PIN TO_ADC1 W DOKUMENTACJI [ ] JESZCZE RAZ SPRAWDZIĆ CZY PINY ADC SĄ DOBRZE PODŁĄCZONE [ ] SPRAWDZIĆ I PODŁĄCZYĆ PIN 5V POD PRZETWORNICĘ"
- note added: "Źródło zasilania +5V i +3.3V"

Commit message: Nucleo-shield pins change
Connections:
- net DETECT_SD: now also U13.1.13 (PA13)
- net SPI_MOSI: now reaches U13.1.45 (PD7)
- net SPI_CLK: now reaches U13.2.11 (PA5)
- net SPI_MISO: now reaches U13.2.13 (PA6)
- net SS_2: now reaches U13.2.16 (PB12)
- net SS_1: now reaches U13.2.17 (PB6)
- net SS_3: now reaches U13.2.18 (PB11)
- net SIG_6: now reaches U13.2.37 (PA3)
Changed lines of the file:
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@@
+	(wire
+		(pts
+			(xy 172.72 92.71) (xy 182.88 92.71)
+		)
+		(stroke
+			(width 0)
+			(type default)
+		)
+	)
 	(wire
 		(pts
@@
 	(wire
 		(pts
+			(xy 93.98 69.85) (xy 99.06 69.85)
+		)
+		(stroke
+			(width 0)
+			(type default)
+		)
+	)
+	(wire
+		(pts
 			(xy 287.02 72.39) (xy 287.02 78.74)
 		)
@@
 	(wire
 		(pts
+			(xy 172.72 105.41) (xy 182.88 105.41)
+		)
+		(stroke
+			(width 0)
+			(type default)
+		)
+	)
+	(wire
+		(pts
 			(xy 351.79 59.69) (xy 351.79 60.96)
 		)
@@
 	(wire
 		(pts
+			(xy 93.98 92.71) (xy 99.06 92.71)
+		)
+		(stroke
+			(width 0)
+			(type default)
+		)
+	)
+	(wire
+		(pts
+			(xy 93.98 173.99) (xy 99.06 173.99)
+		)
+		(stroke
+			(width 0)
+			(type default)
+		)
+	)
+	(wire
+		(pts
 			(xy 358.14 60.96) (xy 358.14 59.69)
 		)
@@
 	(wire
 		(pts
+			(xy 172.72 87.63) (xy 182.88 87.63)
+		)
+		(stroke
+			(width 0)
+			(type default)
+		)
+	)
+	(wire
+		(pts
 			(xy 93.98 64.77) (xy 99.06 64.77)
 		)
@@
 	(wire
 		(pts
-			(xy 93.98 69.85) (xy 99.06 69.85)
-		)
-		(stroke
-			(width 0)
-			(type default)
-		)
-	)
-	(wire
-		(pts
 			(xy 351.79 49.53) (xy 351.79 52.07)
 		)
@@
 	(wire
 		(pts
+			(xy 172.72 153.67) (xy 182.88 153.67)
+		)
+		(stroke
+			(width 0)
+			(type default)
+		)
+	)
+	(wire
+		(pts
 			(xy 358.14 69.85) (xy 358.14 72.39)
 		)
@@
 	(wire
 		(pts
+			(xy 172.72 100.33) (xy 182.88 100.33)
+		)
+		(stroke
+			(width 0)
+			(type default)
+		)
+	)
+	(wire
+		(pts
 			(xy 278.13 90.17) (xy 278.13 92.71)
 		)
@@
 		(pts
 			(xy 388.62 69.85) (xy 388.62 72.39)
+		)
+		(stroke
+			(width 0)
+			(type default)
+		)
+	)
+	(wire
+		(pts
+			(xy 172.72 102.87) (xy 182.88 102.87)
 		)
 		(stroke
@@
 		)
 	)
+	(hierarchical_label "SIG_6"
+		(shape input)
+		(at 182.88 153.67 0)
+		(effects
+			(font
+				(size 1.27 1.27)
+			)
+			(justify left)
+		)
+	)
+	(hierarchical_label "SPI_MOSI"
+		(shape bidirectional)
+		(at 93.98 173.99 180)
+		(effects
+			(font
+				(size 1.27 1.27)
+			)
+			(justify right)
+		)
+	)
+	(hierarchical_label "SS_1"
+		(shape output)
+		(at 182.88 102.87 0)
+		(effects
+			(font
+				(size 1.27 1.27)
+			)
+			(justify left)
+		)
+	)
 	(hierarchical_label "SDMMC_D1"
 		(shape bidirectional)
@@
 		)
 	)
+	(hierarchical_label "SS_2"
+		(shape output)
+		(at 182.88 100.33 0)
+		(effects
+			(font
+				(size 1.27 1.27)
+			)
+			(justify left)
+		)
+	)
+	(hierarchical_label "SPI_CLK"
+		(shape bidirectional)
+		(at 182.88 87.63 0)
+		(effects
+			(font
+				(size 1.27 1.27)
+			)
+			(justify left)
+		)
+	)
+	(hierarchical_label "SPI_MISO"
+		(shape bidirectional)
+		(at 182.88 92.71 0)
+		(effects
+			(font
+				(size 1.27 1.27)
+			)
+			(justify left)
+		)
+	)
 	(hierarchical_label "SIG_3"
 		(shape input)
@@
 	)
 	(hierarchical_label "DETECT_SD"
-		(shape bidirectional)
-		(at 83.82 73.66 180)
+		(shape input)
+		(at 93.98 92.71 180)
 		(effects
 			(font
@@
 		)
 	)
+	(hierarchical_label "SS_3"
+		(shape output)
+		(at 182.88 105.41 0)
+		(effects
+			(font
+				(size 1.27 1.27)
+			)
+			(justify left)
+		)
+	)

Commit message: Layout major change, .gitignore added
Parts:
- added NT1: NetTie_2, NetTie:NetTie-2_SMD_Pad0.5mm, symbol Device:NetTie_2
Connections:
- net GND: now also U13.1.08 (GND), U13.1.49 (GND), U13.1.60 (GND), U13.2.39 (GND), U13.2.54 (GND), U13.2.63 (GND), NT1.1
- net GNDA: now also NT1.2
- no-connect marks 19 -> 27
