File: Nucleo.kicad_sch (KiCad schematic)
At the start: 19 parts, among them U13 Nucleo-H755ZIQ-Morpho, U14 TPS61236PRWLR, U15 LD1117S50TR_SOT223

Commit message: Errors in pcb layout removed, footprints fixed, microvias changed to regular vias
Parts:
- added C48: 10u, Capacitor_SMD:C_0603_1608Metric_Pad1.08x0.95mm_HandSolder, symbol Device:C
Connections:
- net +5V: now also U13.1.06 (5V_EXT), C48.1
- net GND: now also C48.2
- net 3.3V_Nucleo: now reaches U13.1.16 (3V3)
- no-connect marks 27 -> 111
Other:
- note removed: "[x] SIG PONUMEROWAĆ ODPOWIEDNIO Z DOKUMENTACJĄ [x] DODAĆ PIN T0_ADC2 [x] SPRAWDZIĆ PIN TO_ADC1 W DOKUMENTACJI [ ] JESZCZE RAZ SPRAWDZIĆ CZY PINY ADC SĄ DOBRZE PODŁĄCZONE [ ] SPRAWDZIĆ I PODŁĄCZYĆ PIN 5V POD PRZETWORNICĘ"

Commit message: Vias fixed, generated gerber files
Parts:
- U15: value LD1117S50TR_SOT223 -> LD1117S33TR_SOT223
Changed lines of the file:
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@@
 			)
 		)
-		(property "Value" "LD1117S50TR_SOT223"
+		(property "Value" "LD1117S33TR_SOT223"
 			(at 339.09 91.694 0)
 			(show_name no)
@@
 			)
 		)
-		(property "Description" "800mA Fixed Low Drop Positive Voltage Regulator, Fixed Output 5.0V, SOT-223"
+		(property "Description" "800mA Fixed Low Drop Positive Voltage Regulator, Fixed Output 3.3V, SOT-223"
 			(at 327.66 85.09 0)
 			(hide yes)
