File: Uklad_wzmacniaczy.kicad_sch (KiCad schematic)
At the start: 88 parts, among them J1 SJ1-3523N, J2 MEM2080-00-128-00-A, J3 Conn_01x10_Pin, U1 OPA2388IDR, U10 AD5162BRMZ10-RL7, U11 AD5162BRMZ10-RL7, U12 LT3094EMSE-TRPBF, U2 REF2033QDDCRQ1, U3 AD8421ARMZ, U4 OPA388IDR, U5 AD8421ARMZ, U6 TPD4E1B06DRLR, U7 AD5162BRMZ10-RL7, U8 LT3042EMSE-TRPBF, U9 TPS65135RTER

Commit message: Vias fixed, generated gerber files
Parts:
- R10, R4: value 200-400k -> 220k
Other:
- note added: "Rezystor 200k do 400k"
Changed lines of the file:
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@@
 		)
 	)
+	(text "Rezystor 200k do 400k"
+		(exclude_from_sim no)
+		(at 273.558 67.31 0)
+		(effects
+			(font
+				(size 1.27 1.27)
+			)
+		)
+	)
 	(text "Test points"
 		(exclude_from_sim no)
@@
 		)
 	)
+	(text "Rezystor 200k do 400k"
+		(exclude_from_sim no)
+		(at 297.688 111.252 0)
+		(effects
+			(font
+				(size 1.27 1.27)
+			)
+		)
+	)
 	(junction
 		(at 250.19 40.64)
@@
 			)
 		)
-		(property "Value" "200-400k"
+		(property "Value" "220k"
 			(at 296.926 122.428 0)
 			(show_name no)
@@
 			)
 		)
-		(property "Value" "200-400k"
+		(property "Value" "220k"
 			(at 261.366 70.358 0)
 			(show_name no)

Commit message: Minor fixes
Parts:
- R10, R4: value 220k -> 10k
- R12, R15: value 49.9k -> 45.3k
Connections:
- net +5VA renamed +4.5VA
- net -5VA renamed -4.5VA
Other:
- note added: "Stabilizator napięcia +4.5V"
- note added: "Stabilizator napięcia -4.5V"
- note removed: "Stabilizator napięcia +5V"
- note removed: "Stabilizator napięcia -5V"
